Commit message: updates to model to work with director distro

File: models/anymal_description/model_pre_argos.urdf (robot description, URDF)
Before this commit: robot anymal, 28 links, 27 joints
Links:
- link LF_HIP: geometry collision cylinder length=0.08 radius=0.04; visual mesh filename=/home/mfallon/rpg-navigation/code_externals/models/anymal_d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 scale=0.001 0.001 0.001
- link LF_SHANK: geometry collision cylinder length=0.13 radius=0.015; collision cylinder length=0.19 radius=0.015
- link LF_THIGH: geometry collision cylinder length=0.08 radius=0.04; collision cylinder length=0.2 radius=0.01
- link LH_HIP: geometry collision cylinder length=0.08 radius=0.04; visual mesh filename=/home/mfallon/rpg-navigation/code_externals/models/anymal_d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 scale=0.001 0.001 0.001
- link LH_SHANK: geometry collision cylinder length=0.13 radius=0.015; collision cylinder length=0.19 radius=0.015
- link LH_THIGH: geometry collision cylinder length=0.08 radius=0.04; collision cylinder length=0.2 radius=0.01
- link RF_HIP: geometry collision cylinder length=0.08 radius=0.04; visual mesh filename=/home/mfallon/rpg-navigation/code_externals/models/anymal_d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 scale=0.001 0.001 0.001
- link RF_SHANK: geometry collision cylinder length=0.13 radius=0.015; collision cylinder length=0.19 radius=0.015
- link RF_THIGH: geometry collision cylinder length=0.08 radius=0.04; collision cylinder length=0.2 radius=0.01
- link RH_HIP: geometry collision cylinder length=0.08 radius=0.04; visual mesh filename=/home/mfallon/rpg-navigation/code_externals/models/anymal_d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 scale=0.001 0.001 0.001
- link RH_SHANK: geometry collision cylinder length=0.13 radius=0.015; collision cylinder length=0.19 radius=0.015
- link RH_THIGH: geometry collision cylinder length=0.08 radius=0.04; collision cylinder length=0.2 radius=0.01
- link base: geometry collision box size=0.5 0.18 0.26; collision box size=0.77 0.18 0.03
