Commit message: clean up the path using luke's suggestion
change urdf to point to _ori descriptions

File: models/anymal_description/model_laser.urdf (robot description, URDF)
Before this commit: robot anymal, 33 links, 32 joints
Links:
- link LF_FOOT_SENSOR: geometry collision sphere radius=0.02; visual mesh filename=package://anymal_description_ori/urdf/foot/anymal_foot_2.dae scale=0.001 0.001 0.001
- link LF_HIP: geometry collision cylinder length=0.08 radius=0.04; visual mesh filename=package://anymal_description_ori/urdf/hip/anymal_hip_l.dae scale=0.001 0.001 0.001
- link LF_SHANK: geometry collision cylinder length=0.13 radius=0.015; collision cylinder length=0.19 radius=0.015
- link LF_THIGH: geometry collision cylinder length=0.08 radius=0.04; collision cylinder length=0.2 radius=0.01
- link LH_FOOT_SENSOR: geometry collision sphere radius=0.02; visual mesh filename=package://anymal_description_ori/urdf/foot/anymal_foot_2.dae scale=0.001 0.001 0.001
- link LH_HIP: geometry collision cylinder length=0.08 radius=0.04; visual mesh filename=package://anymal_description_ori/urdf/hip/anymal_hip_r.dae scale=0.001 0.001 0.001
- link LH_SHANK: geometry collision cylinder length=0.13 radius=0.015; collision cylinder length=0.19 radius=0.015
- link LH_THIGH: geometry collision cylinder length=0.08 radius=0.04; collision cylinder length=0.2 radius=0.01
- link RF_FOOT_SENSOR: geometry collision sphere radius=0.02; visual mesh filename=package://anymal_description_ori/urdf/foot/anymal_foot_2.dae scale=0.001 0.001 0.001
- link RF_HIP: geometry collision cylinder length=0.08 radius=0.04; visual mesh filename=package://anymal_description_ori/urdf/hip/anymal_hip_r.dae scale=0.001 0.001 0.001
- link RF_SHANK: geometry collision cylinder length=0.13 radius=0.015; collision cylinder length=0.19 radius=0.015
- link RF_THIGH: geometry collision cylinder length=0.08 radius=0.04; collision cylinder length=0.2 radius=0.01
- link RH_FOOT_SENSOR: geometry collision sphere radius=0.02; visual mesh filename=package://anymal_description_ori/urdf/foot/anymal_foot_2.dae scale=0.001 0.001 0.001
- link RH_HIP: geometry collision cylinder length=0.08 radius=0.04; visual mesh filename=package://anymal_description_ori/urdf/hip/anymal_hip_l.dae scale=0.001 0.001 0.001
- link RH_SHANK: geometry collision cylinder length=0.13 radius=0.015; collision cylinder length=0.19 radius=0.015
- link RH_THIGH: geometry collision cylinder length=0.08 radius=0.04; collision cylinder length=0.2 radius=0.01
- link actuated_lidar_front_dynamixel_axis_aligned: geometry visual mesh filename=package://actuated_lidar_description_ori/mesh/case_fix.dae scale=.001 .001 .001; visual mesh filename=package://dynamixel_description/mesh/MX64.stl scale=.001 .001 .001
- link actuated_lidar_front_hokuyo: geometry collision cylinder length=0.12 radius=0.06; visual mesh filename=package://actuated_lidar_description_ori/mesh/case_moving.d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 scale=.001 .001 .001
- link base: geometry collision box size=0.1 0.1 0.07; collision box size=0.1 0.1 0.07

File: models/anymal_description/model_laser_drake.urdf (robot description, URDF)
Before this commit: robot anymal, 33 links, 32 joints
Links:
- link LF_FOOT_SENSOR: geometry collision sphere radius=0.02; visual mesh filename=package://anymal_description_ori/urdf/foot/anymal_foot_2.dae scale=0.001 0.001 0.001
- link LF_HIP: geometry collision cylinder length=0.08 radius=0.04; visual mesh filename=package://anymal_description_ori/urdf/hip/anymal_hip_l.dae scale=0.001 0.001 0.001
- link LF_SHANK: geometry collision cylinder length=0.13 radius=0.015; collision cylinder length=0.19 radius=0.015
- link LF_THIGH: geometry collision cylinder length=0.08 radius=0.04; collision cylinder length=0.2 radius=0.01
- link LH_FOOT_SENSOR: geometry collision sphere radius=0.02; visual mesh filename=package://anymal_description_ori/urdf/foot/anymal_foot_2.dae scale=0.001 0.001 0.001
- link LH_HIP: geometry collision cylinder length=0.08 radius=0.04; visual mesh filename=package://anymal_description_ori/urdf/hip/anymal_hip_r.dae scale=0.001 0.001 0.001
- link LH_SHANK: geometry collision cylinder length=0.13 radius=0.015; collision cylinder length=0.19 radius=0.015
- link LH_THIGH: geometry collision cylinder length=0.08 radius=0.04; collision cylinder length=0.2 radius=0.01
- link RF_FOOT_SENSOR: geometry collision sphere radius=0.02; visual mesh filename=package://anymal_description_ori/urdf/foot/anymal_foot_2.dae scale=0.001 0.001 0.001
- link RF_HIP: geometry collision cylinder length=0.08 radius=0.04; visual mesh filename=package://anymal_description_ori/urdf/hip/anymal_hip_r.dae scale=0.001 0.001 0.001
- link RF_SHANK: geometry collision cylinder length=0.13 radius=0.015; collision cylinder length=0.19 radius=0.015
- link RF_THIGH: geometry collision cylinder length=0.08 radius=0.04; collision cylinder length=0.2 radius=0.01
- link RH_FOOT_SENSOR: geometry collision sphere radius=0.02; visual mesh filename=package://anymal_description_ori/urdf/foot/anymal_foot_2.dae scale=0.001 0.001 0.001
- link RH_HIP: geometry collision cylinder length=0.08 radius=0.04; visual mesh filename=package://anymal_description_ori/urdf/hip/anymal_hip_l.dae scale=0.001 0.001 0.001
- link RH_SHANK: geometry collision cylinder length=0.13 radius=0.015; collision cylinder length=0.19 radius=0.015
- link RH_THIGH: geometry collision cylinder length=0.08 radius=0.04; collision cylinder length=0.2 radius=0.01
- link actuated_lidar_front_dynamixel_axis_aligned: geometry visual mesh filename=package://actuated_lidar_description_ori/mesh/case_fix.dae scale=.001 .001 .001; visual mesh filename=package://dynamixel_description/mesh/MX64.stl scale=.001 .001 .001
- link actuated_lidar_front_hokuyo: geometry collision cylinder length=0.12 radius=0.06; visual mesh filename=package://actuated_lidar_description_ori/mesh/case_moving.d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 scale=.001 .001 .001
- link base: geometry collision box size=0.1 0.1 0.07; collision box size=0.1 0.1 0.07

Commit message: undo changes to we have one location for meshes

File: models/anymal_description/model_laser.urdf (robot description, URDF)
Before this commit: robot anymal, 33 links, 32 joints
Links:
- link LF_FOOT_SENSOR: geometry collision sphere radius=0.02; visual mesh filename=package://anymal_description/urdf/foot/anymal_foot_2.dae scale=0.001 0.001 0.001
- link LF_HIP: geometry collision cylinder length=0.08 radius=0.04; visual mesh filename=package://anymal_description/urdf/hip/anymal_hip_l.dae scale=0.001 0.001 0.001
- link LF_SHANK: geometry collision cylinder length=0.13 radius=0.015; collision cylinder length=0.19 radius=0.015
- link LF_THIGH: geometry collision cylinder length=0.08 radius=0.04; collision cylinder length=0.2 radius=0.01
- link LH_FOOT_SENSOR: geometry collision sphere radius=0.02; visual mesh filename=package://anymal_description/urdf/foot/anymal_foot_2.dae scale=0.001 0.001 0.001
- link LH_HIP: geometry collision cylinder length=0.08 radius=0.04; visual mesh filename=package://anymal_description/urdf/hip/anymal_hip_r.dae scale=0.001 0.001 0.001
- link LH_SHANK: geometry collision cylinder length=0.13 radius=0.015; collision cylinder length=0.19 radius=0.015
- link LH_THIGH: geometry collision cylinder length=0.08 radius=0.04; collision cylinder length=0.2 radius=0.01
- link RF_FOOT_SENSOR: geometry collision sphere radius=0.02; visual mesh filename=package://anymal_description/urdf/foot/anymal_foot_2.dae scale=0.001 0.001 0.001
- link RF_HIP: geometry collision cylinder length=0.08 radius=0.04; visual mesh filename=package://anymal_description/urdf/hip/anymal_hip_r.dae scale=0.001 0.001 0.001
- link RF_SHANK: geometry collision cylinder length=0.13 radius=0.015; collision cylinder length=0.19 radius=0.015
- link RF_THIGH: geometry collision cylinder length=0.08 radius=0.04; collision cylinder length=0.2 radius=0.01
- link RH_FOOT_SENSOR: geometry collision sphere radius=0.02; visual mesh filename=package://anymal_description/urdf/foot/anymal_foot_2.dae scale=0.001 0.001 0.001
- link RH_HIP: geometry collision cylinder length=0.08 radius=0.04; visual mesh filename=package://anymal_description/urdf/hip/anymal_hip_l.dae scale=0.001 0.001 0.001
- link RH_SHANK: geometry collision cylinder length=0.13 radius=0.015; collision cylinder length=0.19 radius=0.015
- link RH_THIGH: geometry collision cylinder length=0.08 radius=0.04; collision cylinder length=0.2 radius=0.01
- link actuated_lidar_front_dynamixel_axis_aligned: geometry visual mesh filename=package://actuated_lidar_description/mesh/case_fix.dae scale=.001 .001 .001; visual mesh filename=package://dynamixel_description/mesh/MX64.stl scale=.001 .001 .001
- link actuated_lidar_front_hokuyo: geometry collision cylinder length=0.12 radius=0.06; visual mesh filename=package://actuated_lidar_description/mesh/case_moving.dae scale=.001 .001 .001
- link base: geometry collision box size=0.1 0.1 0.07; collision box size=0.1 0.1 0.07

File: models/anymal_description/model_laser_drake.urdf (robot description, URDF)
Before this commit: robot anymal, 33 links, 32 joints
Links:
- link LF_FOOT_SENSOR: geometry collision sphere radius=0.02; visual mesh filename=package://anymal_description/urdf/foot/anymal_foot_2.dae scale=0.001 0.001 0.001
- link LF_HIP: geometry collision cylinder length=0.08 radius=0.04; visual mesh filename=package://anymal_description/urdf/hip/anymal_hip_l.dae scale=0.001 0.001 0.001
- link LF_SHANK: geometry collision cylinder length=0.13 radius=0.015; collision cylinder length=0.19 radius=0.015
- link LF_THIGH: geometry collision cylinder length=0.08 radius=0.04; collision cylinder length=0.2 radius=0.01
- link LH_FOOT_SENSOR: geometry collision sphere radius=0.02; visual mesh filename=package://anymal_description/urdf/foot/anymal_foot_2.dae scale=0.001 0.001 0.001
- link LH_HIP: geometry collision cylinder length=0.08 radius=0.04; visual mesh filename=package://anymal_description/urdf/hip/anymal_hip_r.dae scale=0.001 0.001 0.001
- link LH_SHANK: geometry collision cylinder length=0.13 radius=0.015; collision cylinder length=0.19 radius=0.015
- link LH_THIGH: geometry collision cylinder length=0.08 radius=0.04; collision cylinder length=0.2 radius=0.01
- link RF_FOOT_SENSOR: geometry collision sphere radius=0.02; visual mesh filename=package://anymal_description/urdf/foot/anymal_foot_2.dae scale=0.001 0.001 0.001
- link RF_HIP: geometry collision cylinder length=0.08 radius=0.04; visual mesh filename=package://anymal_description/urdf/hip/anymal_hip_r.dae scale=0.001 0.001 0.001
- link RF_SHANK: geometry collision cylinder length=0.13 radius=0.015; collision cylinder length=0.19 radius=0.015
- link RF_THIGH: geometry collision cylinder length=0.08 radius=0.04; collision cylinder length=0.2 radius=0.01
- link RH_FOOT_SENSOR: geometry collision sphere radius=0.02; visual mesh filename=package://anymal_description/urdf/foot/anymal_foot_2.dae scale=0.001 0.001 0.001
- link RH_HIP: geometry collision cylinder length=0.08 radius=0.04; visual mesh filename=package://anymal_description/urdf/hip/anymal_hip_l.dae scale=0.001 0.001 0.001
- link RH_SHANK: geometry collision cylinder length=0.13 radius=0.015; collision cylinder length=0.19 radius=0.015
- link RH_THIGH: geometry collision cylinder length=0.08 radius=0.04; collision cylinder length=0.2 radius=0.01
- link actuated_lidar_front_dynamixel_axis_aligned: geometry visual mesh filename=package://actuated_lidar_description/mesh/case_fix.dae scale=.001 .001 .001; visual mesh filename=package://dynamixel_description/mesh/MX64.stl scale=.001 .001 .001
- link actuated_lidar_front_hokuyo: geometry collision cylinder length=0.12 radius=0.06; visual mesh filename=package://actuated_lidar_description/mesh/case_moving.dae scale=.001 .001 .001
- link base: geometry collision box size=0.1 0.1 0.07; collision box size=0.1 0.1 0.07
