Commit message: add bits and pieces for the other robots in director

File: models/hyq_description/robots/hyq.urdf (robot description, URDF)
Before this commit: robot hyq, 44 links, 43 joints
Links:
- link asus_mount_link: geometry collision box size=0.05 .18 0.035; visual mesh filename=package://hyq_description/meshes/sensors/asus_xtion.dae scale=1 1 1
- link laser_mount_link: geometry visual mesh filename=package://hyq_description/meshes/hokuyo_utm30lx/hokuyo_utm_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 scale=0.0254 0.0254 0.0254
