Commit message: update some configs to multisense on husky

File: models/husky_description/model.urdf (robot description, URDF)
Before this commit: robot husky_robot, 34 links, 33 joints
Joints:
- removed joint multisense_to_ptu
- added joint head_joint: type fixed, parent base_link, child head_root, origin xyz=0.315 0.0 0.593
- joint ptu_pan: type revolute -> fixed
- joint ptu_tilt: type revolute -> fixed
